Commit message: change from continous to revol for joint 1 4 6

File: src/pick_and_place/urdf/kinova_6dof_sim.urdf (robot description, URDF)
Before this commit: robot gen3, 10 links, 9 joints
Joints:
- joint joint_1: limit effort=39 velocity=1.3963 -> lower=-2.97 upper=2.97 effort=39 velocity=1.3963; type continuous -> revolute
- joint joint_4: limit effort=9 velocity=1.2218 -> lower=-3.14 upper=3.14 effort=9 velocity=1.2218; type continuous -> revolute
- joint joint_6: limit effort=9 velocity=1.2218 -> lower=-3.14 upper=3.14 effort=9 velocity=1.2218; type continuous -> revolute
